File: Motherboards/SHVC-CPU-01/Rev A/SHVC-CPU-01-Back.kicad_sch (KiCad schematic)
At the start: 458 parts, among them P2 11 Pin FFC Connector, Q1 C4699, Q10 C2412, Q11 C2412, Q12 C2412, Q13 C2412, Q14 C2412, Q15 C2412, Q16 C2412, Q17 C2412, Q18 C2412, Q2 C4699, Q3 A1037, Q4 A1037, Q5 A1037, Q6 A1037, Q7 A1037, Q8 A1037, Q9 C2412, X1 21.47727Mhz

Commit message: Fix Transistor Symbols in SHVC-CPU-01 Schematic
While wired correctly, these were visually borked in the
schematic because of my visual oriented style. I made custom
symbols to accomodate when correcting.

Thanks RGBeter for reporting this issue.
Parts:
- Q1, Q2: symbol Transistor_BJT:Q_NPN_EBC -> OpenSFC:Q_NPN_BEC
- Q10, Q11, Q12, Q13, Q14, Q15, Q16, Q17, Q18, Q9: footprint OpenSFC:Q_SOT -> OpenSFC:Q_SOT_PNP_EBC; symbol Transistor_BJT:Q_NPN_EBC -> OpenSFC:Q_PNP_EBC
- Q3, Q4, Q5, Q6, Q7, Q8: footprint OpenSFC:Q_SOT -> OpenSFC:Q_SOT_PNP_EBC; symbol Transistor_BJT:Q_PNP_BEC -> OpenSFC:Q_PNP_EBC
Connections:
- net +5V: now also Q10.3 (E), Q11.3 (E), Q12.3 (E), Q9.3 (E); no longer Q10.2 (B), Q11.2 (B), Q12.2 (B), Q9.2 (B)
- net +9V: now also Q16.3 (E), Q17.3 (E); no longer Q16.2 (B), Q17.2 (B)
- net +9VS: now also Q18.3 (E); no longer Q18.2 (B)
- net C57+: now also Q10.1 (C); no longer Q10.3 (C)
- net C59+: now also Q11.1 (C); no longer Q11.3 (C)
- net GND: now also Q13.1 (C), Q3.3 (E), Q4.3 (E), Q5.3 (E), Q6.3 (E), Q7.3 (E), Q8.3 (E); no longer Q13.3 (C), Q3.1 (B), Q4.1 (B), Q5.1 (B), Q6.1 (B), Q7.1 (B), Q8.1 (B)
- net II1: now also Q15.1 (C); no longer Q15.3 (C)
- net II2: now also Q14.1 (C); no longer Q14.3 (C)
- net OUT1: now also Q15.3 (E), Q17.2 (B); no longer Q15.2 (B), Q17.1 (E)
- net OUT2: now also Q14.3 (E), Q16.2 (B); no longer Q14.2 (B), Q16.1 (E)
- net Q13: now also Q13.3 (E); no longer Q13.2 (B)
- net Q14: now also Q14.2 (B); no longer Q14.1 (E)
- net Q18: now also Q18.2 (B); no longer Q18.3 (C)
- net R12: now also Q5.1 (C); no longer Q5.3 (C)
- net R17: now also Q7.1 (C); no longer Q7.3 (C)
- net R7: now also Q3.1 (C); no longer Q3.3 (C)
- net R71: now also Q17.1 (C); no longer Q17.3 (C)
- net at R24.1, R25.2, TP23.1: now also Q9.1 (C); no longer Q9.3 (C)
- net at R58.1, R66.2, R67.2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: now also Q16.1 (C); no longer Q16.3 (C)
- net at C12.1, R30.1, R31.2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: now also Q10.2 (B); no longer Q10.1 (E)
- net at R13.2, R15.2, TP35.1: now also Q6.1 (C); no longer Q6.3 (C)
- net at C54.2, R59.2, TP72.1: now also Q15.2 (B); no longer Q15.1 (E)
- net at C19.1, R43.1, R44.1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: now also Q12.2 (B); no longer Q12.1 (E)
- net at R10.1, R8.2, TP29.1: now also Q4.1 (C); no longer Q4.3 (C)
- net at C17.2, R100.1, R38.1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: now also Q11.2 (B); no longer Q11.1 (E)
- net at R18.1, R20.1, TP37.1: now also Q8.1 (C); no longer Q8.3 (C)
- net at R48.1, TP75.1: now also Q13.2 (B); no longer Q13.1 (E)
- net at C20.2, R45.2, TP52.1: now also Q12.1 (C); no longer Q12.3 (C)
- net at R22.1, R23.1, TP50.1: now also Q9.2 (B); no longer Q9.1 (E)

Commit message: Also correct the audio transistor symbols
Same issue as with the ones in the previous fix, wiring was
correct but the schematic symbol was wrong.
Parts:
- Q1, Q2: footprint OpenSFC:Q_SOT -> OpenSFC:Q_SOT_NPM_BEC
- Q10: footprint OpenSFC:Q_SOT_PNP_EBC -> OpenSFC:Q_SOT_NPM_BEC_Alt
- Q11, Q12, Q13, Q14, Q15, Q16, Q17, Q18, Q9: footprint OpenSFC:Q_SOT_PNP_EBC -> OpenSFC:Q_SOT_NPM_BEC_Alt; symbol OpenSFC:Q_PNP_EBC -> OpenSFC:Q_NPN_BEC_Alt
Connections:
- net GND: now also Q1.2 (E), Q2.2 (E); no longer Q1.3 (C), Q2.3 (C)
- net TC.2: now also Q1.3 (C); no longer Q1.2 (E)
- net at R5.1, R6.1, TP214.1: now also Q2.3 (C); no longer Q2.2 (E)
Changed lines of the file:
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@@
 	(title_block
 		(title "SHVC-CPU-01")
-		(date "2025-10-27")
-		(rev "A (SP1)")
+		(date "2025-10-30")
+		(rev "A (SP2)")
 		(company "License: CERN-OHL-S")
 		(comment 1 "This Document Is Not Endorsed By Nintendo")
@@
 	)
 	(symbol
-		(lib_id "OpenSFC:Q_PNP_EBC")
+		(lib_id "OpenSFC:Q_NPN_BEC_Alt")
 		(at 96.52 220.98 0)
 		(unit 1)
@@
 			)
 		)
-		(property "Footprint" "OpenSFC:Q_SOT_PNP_EBC"
+		(property "Footprint" "OpenSFC:Q_SOT_NPM_BEC_Alt"
 			(at 96.52 220.98 0)
 			(effects
@@
 			)
 		)
-		(property "Footprint" "OpenSFC:Q_SOT"
+		(property "Footprint" "OpenSFC:Q_SOT_NPM_BEC"
 			(at 490.22 577.85 0)
 			(effects
@@
 	)
 	(symbol
-		(lib_id "OpenSFC:Q_PNP_EBC")
+		(lib_id "OpenSFC:Q_NPN_BEC_Alt")
 		(at 156.21 223.52 0)
 		(unit 1)
@@
 			)
 		)
-		(property "Footprint" "OpenSFC:Q_SOT_PNP_EBC"
+		(property "Footprint" "OpenSFC:Q_SOT_NPM_BEC_Alt"
 			(at 156.21 223.52 0)
 			(effects
@@
 	)
 	(symbol
-		(lib_id "OpenSFC:Q_PNP_EBC")
+		(lib_id "OpenSFC:Q_NPN_BEC_Alt")
 		(at 335.28 124.46 0)
 		(unit 1)
@@
 			)
 		)
-		(property "Footprint" "OpenSFC:Q_SOT_PNP_EBC"
+		(property "Footprint" "OpenSFC:Q_SOT_NPM_BEC_Alt"
 			(at 335.28 124.46 0)
 			(effects
@@
 	)
 	(symbol
-		(lib_id "OpenSFC:Q_PNP_EBC")
+		(lib_id "OpenSFC:Q_NPN_BEC_Alt")
 		(at 425.45 165.1 0)
 		(unit 1)
@@
 			)
 		)
-		(property "Footprint" "OpenSFC:Q_SOT_PNP_EBC"
+		(property "Footprint" "OpenSFC:Q_SOT_NPM_BEC_Alt"
 			(at 425.45 165.1 0)
 			(effects
@@
 			)
 		)
-		(property "Footprint" "OpenSFC:Q_SOT"
+		(property "Footprint" "OpenSFC:Q_SOT_NPM_BEC"
 			(at 480.06 589.28 0)
 			(effects
@@
 	)
 	(symbol
-		(lib_id "OpenSFC:Q_PNP_EBC")
+		(lib_id "OpenSFC:Q_NPN_BEC_Alt")
 		(at 107.95 128.27 0)
 		(unit 1)
@@
 			)
 		)
-		(property "Footprint" "OpenSFC:Q_SOT_PNP_EBC"
+		(property "Footprint" "OpenSFC:Q_SOT_NPM_BEC_Alt"
 			(at 107.95 128.27 0)
 			(effects
@@
 	)
 	(symbol
-		(lib_id "OpenSFC:Q_PNP_EBC")
+		(lib_id "OpenSFC:Q_NPN_BEC_Alt")
 		(at 294.64 114.3 0)
 		(unit 1)
@@
 			)
 		)
-		(property "Footprint" "OpenSFC:Q_SOT_PNP_EBC"
+		(property "Footprint" "OpenSFC:Q_SOT_NPM_BEC_Alt"
 			(at 294.64 114.3 0)
 			(effects
@@
 	)
 	(symbol
-		(lib_id "OpenSFC:Q_PNP_EBC")
+		(lib_id "OpenSFC:Q_NPN_BEC_Alt")
 		(at 74.93 220.98 0)
 		(unit 1)
@@
 			)
 		)
-		(property "Footprint" "OpenSFC:Q_SOT_PNP_EBC"
+		(property "Footprint" "OpenSFC:Q_SOT_NPM_BEC_Alt"
 			(at 74.93 220.98 0)
 			(effects
@@
 	)
 	(symbol
-		(lib_id "OpenSFC:Q_PNP_EBC")
+		(lib_id "OpenSFC:Q_NPN_BEC_Alt")
 		(at 125.73 128.27 0)
 		(unit 1)
@@
 			)
 		)
-		(property "Footprint" "OpenSFC:Q_SOT_PNP_EBC"
+		(property "Footprint" "OpenSFC:Q_SOT_NPM_BEC_Alt"
 			(at 125.73 128.27 0)
 			(effects
@@
 			)
 		)
-		(property "Footprint" "OpenSFC:Q_SOT_PNP_EBC"
+		(property "Footprint" "OpenSFC:Q_SOT_NPM_BEC_Alt"
 			(at 398.78 76.2 0)
 			(effects
@@
 	)
 	(symbol
-		(lib_id "OpenSFC:Q_PNP_EBC")
+		(lib_id "OpenSFC:Q_NPN_BEC_Alt")
 		(at 326.39 111.76 0)
 		(unit 1)
@@
 			)
 		)
-		(property "Footprint" "OpenSFC:Q_SOT_PNP_EBC"
+		(property "Footprint" "OpenSFC:Q_SOT_NPM_BEC_Alt"
 			(at 326.39 111.76 0)
 			(effects
